File: v2/pcb/mp3-xiao/mp3-xiao.kicad_pcb (KiCad board)
At the start: 2 copper layers, 62 x 45.7 mm, 10 parts, among them SW1 SW_Push, SW2 SW_Push, SW3 SW_Push, U1 OLED ssd1306, U2 ESP32 S3 XIAO, U3 micro sdcard module, U4 PCM5102A

Commit message: worked on v2 pcb
Parts:
- added SW4: SW_Nidec_CAS-120A1, custom_footprint_library:spdt slide switch, F.Cu at (169.0, 105.0)
- added U5: ~, custom_footprint_library:battery_pads, F.Cu at (170.0, 107.0)
- moved SW1 1.06 mm to (118.4, 88.2)
- moved U1 0.67 mm to (142.8, 82.2)
- moved U4 0.11 mm to (148.1, 104.0)
Routing:
- net +3.3V: track 125.7 -> 0.00 mm
- net GND: track 108.9 -> 0.00 mm, vias 4 -> 0
- net Net-(U2-GPIO1): track 85.2 -> 0.00 mm, vias 1 -> 0
- net Net-(U1-SDA): track 62.1 -> 0.00 mm, vias 2 -> 0
- net Net-(U1-SCL): track 56.7 -> 0.00 mm, vias 2 -> 0
- net Net-(U2-GPIO43): track 43.9 -> 0.00 mm, vias 1 -> 0
- net Net-(U2-GPIO9): track 38.1 -> 0.00 mm, vias 1 -> 0
- net Net-(U2-GPIO44): track 28.5 -> 0.00 mm, vias 3 -> 0
- net Net-(U2-GPIO8): track 28.3 -> 0.00 mm, vias 3 -> 0
- net Net-(U2-GPIO7): track 28.3 -> 0.00 mm, vias 3 -> 0
- net Net-(U2-GPIO4): track 25.6 -> 0.00 mm, vias 2 -> 0
- net Net-(U2-GPIO3): track 23.7 -> 0.00 mm, vias 3 -> 0
- net Net-(U2-GPIO2): track 21.2 -> 0.00 mm
