File: v2/pcb/mp3-xiao/mp3-xiao.kicad_sch (KiCad schematic)
At the start: 10 parts, among them SW1 SW_Push, SW2 SW_Push, SW3 SW_Push, U1 OLED ssd1306, U2 ESP32 S3 XIAO, U3 micro sdcard module, U4 PCM5102A

Commit message: worked on v2 pcb
Parts:
- added BT1: Battery_Cell, symbol Device:Battery_Cell
- added SW4: SW_Nidec_CAS-120A1, custom_footprint_library:spdt slide switch, symbol Switch:SW_Nidec_CAS-120A1
- added U5: ~, custom_footprint_library:battery_pads, symbol custom_parts_library:battery_pads
Connections:
- new net: SW4.2 (B), U5.1 (+)
- new net: BT1.2 (-), U5.2 (-)
- new net: BT1.1 (+), SW4.3 (A)
- no-connect marks 2 -> 3
